File: KiCAD_files/spin.kicad_sch (KiCad schematic)
At the start: 48 parts, among them J1 OwnTech_SPIN, J5 FTSH-107-01-F-DV-K, J6 USB_C_Receptacle_USB2.0, SW1 Push Button, SW2 Push Button, T1 Tab, T2 Tab, T3 Tab, T4 Tab, U1 STM32G474RE, U2 AZ1117-33, U3 WE-TVS-82400102, Y1 ECS-240-8-37-CKM-TR3 - 24MHz

Commit message: Minor SPIN revision, bumping to v1.2.1 - Silkscreen improvements.
Signed-off-by: Jean Alinei <jean.alinei@owntech.org>
Parts:
- added G1: LOGO, Footprints:owntech_mini8, symbol Symbols:LOGO
- J5: value FTSH-107-01-F-DV-K -> FTSH-107-01-F-DV-K
Other:
- note added: "Global nets indicate user-accessible signals."
- note removed: "Global net are used to symbolize user accessible signals"
- title: SPIN V1.2.0 -> SPIN V1.2.1
- moved on the sheet: T1, T2, T3, T4
